File: FocDrive.kicad_sch (KiCad schematic)
At the start: 124 parts, among them SW3 KH-BM2.54-3P, U1 HC-PM254-8.5H-1X6PZ, U10 100nF, U11 10uF, U12 RT9193-33GB, U13 10uF, U14 20Ω, U15 20Ω, U16 32.768kHz, U17 AS5047D-ATSM, U18 118kΩ, U19 MCP2562FDT-E/MF, U2 DRV8320HRTVT, U20 100nF, U21 INA240A1PWR, U22 100nF, U23 INA240A1PWR, U5 STM32G474RBT3, U6 MP1584EN-LF-Z, U7 INA240A1PWR, U8 BSZ0901NSATMA1, U9 BSZ0901NSATMA1, X1 8MHz

Commit message: Second cleanup pass
Parts:
- removed H1, H2, H3, H4: HOLEHOLE COPY, HOLEHOLE, symbol gen:HOLEHOLE_COPY
- removed IDRIVE1, VDS1: 2.54-4P TPGT, SW-SMD_8P-L10.2-W6.2-P2.54-LS9.4, symbol gen:2.54-4P_TPGT
- removed R10: 47k, R0603, symbol gen:47k
- removed R18, R9: 18k, R0603, symbol gen:18k
- removed R19: 75k, R0603, symbol gen:75k
- removed SW3: KH-BM2.54-3P, SW-TH_KH-BM2.54-3P, symbol gen:KH-BM2.54-3P
- removed U1: HC-PM254-8.5H-1X6PZ, HDR-TH_HC-PM254-8.5H-1X6PZ, symbol gen:HC-PM254-8.5H-1X6PZ
- added H1, H2, H3, H4: MountingHole_Pad, symbol Mechanical:MountingHole_Pad
- added J1: Conn_ARM_JTAG_SWD_10, Connector_PinHeader_1.27mm:PinHeader_2x05_P1.27mm_Vertical, symbol Connector:Conn_ARM_JTAG_SWD_10
- added R38: 47k, R0603, symbol gen:47k
- added R9: 75k, R0603, symbol gen:75k
- RESET1: value HX 5.2X5.2X1.5H SWITCH TACTILE -> TACTILE SWITCH
Connections:
- net DVDD is gone; now on net +3.3V: C4.1, D2.2, R6.1, U2.24 (DVDD)
- net VDS is gone; now on an unnamed net: U2.20 (VDS)
- net +3.3V: now also C16.1, U17.11 (VDD), J1.1 (VTref)
- net +5V: no longer C16.1, U17.11 (VDD)
- net GND: now also CAN1.3, PWR1.3, J1.3 (GND), J1.5 (GND), J1.9 (GNDDetect), R9.2; no longer R11.2
- net PHASE1: now also C33.2
- net PHASE2: now also C36.2
- net PHASE3: now also C40.2
- net RESET: now also J1.10 (~{RESET})
- net SWCLK: now also J1.4 (SWCLK/TCK)
- net SWDIO: now also J1.2 (SWDIO/TMS)
- net SWO: now also J1.6 (SWO/TDO)
- net VCC: now also PWR1.4
- net at R27.1, U19.6 (CANL): now also CAN1.1
- net at R27.2, U19.7 (CANH): now also CAN1.2
- net IDRIVE: no longer names the net of U2.19 (IDRIVE)
- net IDRIVE: now also R9.1
- net MODE: no longer names the net of U2.18 (MODE)
- net MODE: now also R38.1
- new net: R11.2, R38.2
- no-connect marks 39 -> 34
Other:
- note added: "12V to 5V Converter"
- note added: "3-Shunt Amplified Current Sensing"
- note added: "5V to 3.3V Converter"
- note added: "CAN Transceiver"
- note added: "Crystal Oscillators"
- note added: "External Encoder"
- note added: "Input Power Supply"
- note added: "Logic Power LED"
- note added: "MOSFET Driver"
- note added: "MOSFETs"
- note added: "Motor Outputs"
- note added: "Motor Power LED"
- note added: "Mount Holes"
- note added: "Onboard Encoder"
- note added: "Programming"
- note added: "Reset Button"
- note added: "STM32 Microcontroller"
- note added: "Status LED"
- note added: "USB Debugger"
- note removed: "12v to 5v power supply"
- note removed: "30V max 75Amp max R_on = 4mOhm Q_gd=3nC"
- note removed: "3x3mm MOSFETs (ex.BSZ0904NSI)"
- note removed: "5/3.3V DVDD selector"
- note removed: "5v to 3.3v converter"
- note removed: "CAN TRANS-RECEIVER"
- note removed: "Current Sense Circuit"
- note removed: "DRV8320H"
- note removed: "Gate driver circuit"
- note removed: "IDRIVE Setting the target gate current directly determining the mosfet rise time our mosfet gate-source charge Q = 3nC rise time = Q/IDRIVE (pp 66) we want the rise time of 50ns IDRIVE = Q/50ns = 0.06A"
- note removed: "IDRIVE config"
- note removed: "INA240A1"
- note removed: "MODE Setting the 3xPWM mode Option for 6xPWM as well pp 31"
- note removed: "MODE config"
- note removed: "Motor output terminal"
- note removed: "STM32 MICRO CONTROLLER"
- note removed: "VDS config"
- note removed: "VDS voltage between SHx and SLx limiting the voltage to limit the current max current 50Amps (t_OCP= 4us impulse) drain-source resistance 5mOhm VDS = 50A*0.005Ohm = 0.25V"
- note removed: "configuration IDRIVE = Tied to AGND 10mA IDRIVE = 18 kΩ ± 5% tied to AGND 30mA IDRIVE = 75 kΩ ± 5% tied to AGND 60mA IDRIVE = Hi-Z 120mA IDRIVE = 75 kΩ ± 5% tied to DVDD 260mA IDRIVE = 18 kΩ ± 5% tied to DVDD 570mA IDRIVE = Tied to DVDD 1000mA"
- note removed: "configuration MODE - 00b = Tied to AGND 6xPWM MODE - 01b= 47 kΩ ± 5% tied to AGND 3xPWM ..."
- note removed: "configuration VDS = Tied to AGND 0.06V VDS = 18 kΩ ± 5% tied to AGND 0.13V VDS = 75 kΩ ± 5% tied to AGND 0.26V VDS = Hi-Z 0.6V ( BEST ) VDS = 75 kΩ ± 5% tied to DVDD 1.13VV VDS = 18 kΩ ± 5% tied to DVDD 1.88"
- note removed: "crystal osclliators"
- note removed: "external encoder"
- note removed: "indicators"
- note removed: "input power supply"
- note removed: "mounting holes"
- note removed: "on-board encoder"
- note removed: "power LED Circuit"
- note removed: "programming headers"
- note removed: "reset button"
- note removed: "usb debegger"
- company: (none) -> 01 Binary
- title: SimpleFOC Drive -> FOC Drive
- moved on the sheet: C1, C10, C11, C12, C13, C14, C15, C16, C17, C18, C19, C2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
