File: FocDrive.kicad_pcb (KiCad board)
At the start: 4 copper layers, 80 x 80 mm, 124 parts, among them SW3 KH-BM2.54-3P, U1 HC-PM254-8.5H-1X6PZ, U10 100nF, U11 10uF, U12 RT9193-33GB, U13 10uF, U14 20Ω, U15 20Ω, U16 32.768kHz, U17 AS5047D-ATSM, U18 118kΩ, U19 MCP2562FDT-E/MF, U2 DRV8320HRTVT, U20 100nF, U21 INA240A1PWR, U22 100nF, U23 INA240A1PWR, U5 STM32G474RBT3, U6 MP1584EN-LF-Z, U7 INA240A1PWR, U8 BSZ0901NSATMA1, U9 BSZ0901NSATMA1, X1 8MHz

Commit message: More minor edits
Parts:
- added J1: Conn_ARM_JTAG_SWD_10, Connector_PinHeader_1.27mm:PinHeader_2x05_P1.27mm_Vertical, F.Cu at (50.8, 40.6)
